File: hardware/quadstep.sch (EAGLE design)
At the start: 133 parts, among them U1 A4983, U2 LM317MABDT, U3 A4983, U4 A4983, U5 A4983

Commit message: prototype v020
Parts:
- C5: value 0.1uF -> 0.1uF/100V
Other:
- note added: "*use PRT-08084"
- note added: "*use PRT-08432"
Changed lines of the file:
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@@
 <part name="C4" library="SparkFun" deviceset="CAP" device="0805" value="1uF"/>
 <part name="GND3" library="SparkFun" deviceset="GND" device=""/>
-<part name="C5" library="SparkFun" deviceset="CAP" device="0402-CAP" value="0.1uF"/>
+<part name="C5" library="SparkFun" deviceset="CAP" device="0402-CAP" value="0.1uF/100V"/>
 <part name="GND4" library="SparkFun" deviceset="GND" device=""/>
 <part name="R3" library="SparkFun" deviceset="TRIMPOT" device="SMD" value="10k"/>
@@
 <text x="152.4" y="5.08" size="1.778" layer="97">Reference design by: SchmalzHaus.com/BigEasyDriver</text>
 <text x="342.9" y="129.54" size="1.778" layer="97">3.3V or 5V</text>
+<text x="251.46" y="121.92" size="1.778" layer="97">*use PRT-08432</text>
+<text x="124.46" y="213.36" size="1.778" layer="97">*use PRT-08084</text>
+<text x="266.7" y="213.36" size="1.778" layer="97">*use PRT-08084</text>
+<text x="266.7" y="213.36" size="1.778" layer="97">*use PRT-08084</text>
+<text x="121.92" y="96.52" size="1.778" layer="97">*use PRT-08084</text>
+<text x="264.16" y="96.52" size="1.778" layer="97">*use PRT-08084</text>
 </plain>
 <instances>

Commit message: v020 proto
-added standoffs for heatsinks
-changed A4988 FP
Parts:
- removed U5: A4983, SparkFun:A4983
- added STANDOFF1, STANDOFF2, STANDOFF3, STANDOFF4: STAND-OFFTIGHT, SparkFun-Electromechanical:STAND-OFFTIGHT
- added U6: A4988, SparkFun-PowerIC:A49831:1
- U1, U3, U4: value A4983 -> A4988; device SparkFun:A4983 -> SparkFun-PowerIC:A49831:1
Connections:
- removed net N$45: R25.2, U5.SENSE1
- new net N$61: R4.2, U6.SENSE1
- net DIR1: now also U6.DIR; no longer U1.DIR
- net DIR2: now also U1.DIR; no longer U5.DIR
- net EN1: now also U6.ENABLE; no longer U1.ENABLE
- net EN2: now also U1.ENABLE; no longer U5.ENABLE
- net GND: now also U6.GND@1, U6.GND@2, U6.GND_PAD; no longer U5.GND@1, U5.GND@2, U5.GND_PAD
- net MS11: now also U6.MS1; no longer U1.MS1
- net MS12: now also U1.MS1; no longer U5.MS1
- net MS21: now also U6.MS2; no longer U1.MS2
- net MS22: now also U1.MS2; no longer U5.MS2
- net MS31: now also U6.MS3; no longer U1.MS3
- net MS32: now also U1.MS3; no longer U5.MS3
- net N$10: now also U6.VCP; no longer U1.VCP
- net N$11: now also U6.VREG; no longer U1.VREG
- net N$12: now also U6.ROSC; no longer U1.ROSC
- net N$13: now also U6.CP1; no longer U1.CP1
- net N$14: now also U6.REF; no longer U1.REF
- net N$15: now also U6.CP2; no longer U1.CP2
- net N$3: now also U6.OUT1A; no longer U1.OUT1A
- net N$41: now also U1.OUT1B; no longer U5.OUT1B
- net N$46: now also U1.SENSE2; no longer U5.SENSE2
- net N$47: now also U1.VCP; no longer U5.VCP
- net N$48: now also U1.VREG; no longer U5.VREG
- net N$49: now also U1.ROSC; no longer U5.ROSC
- net N$50: now also U1.REF; no longer U5.REF
- net N$51: now also U1.CP1; no longer U5.CP1
- net N$52: now also U1.CP2; no longer U5.CP2
- net N$54: now also U6.OUT1B; no longer U1.OUT1B
- net N$55: now also U1.OUT1A; no longer U5.OUT1A
- net N$56: now also U1.OUT2A; no longer U5.OUT2A
- net N$57: now also U1.OUT2B; no longer U5.OUT2B
- net N$6: now also U6.OUT2A; no longer U1.OUT2A
- net N$7: now also U6.OUT2B; no longer U1.OUT2B
- net N$8: now also R25.2; no longer R4.2
- net N$9: now also U6.SENSE2; no longer U1.SENSE2
- net RST1: now also U6.RESET; no longer U1.RESET
- net RST2: now also U1.RESET; no longer U5.RESET
- net SLP1: now also U6.SLEEP; no longer U1.SLEEP
- net SLP2: now also U1.SLEEP; no longer U5.SLEEP
- net STP1: now also U6.STEP; no longer U1.STEP
- net STP2: now also U1.STEP; no longer U5.STEP
- net VCC: now also U6.VDD; no longer U5.VDD
- net VIN: now also U6.VBB1, U6.VBB2; no longer U5.VBB1, U5.VBB2
Other:
- moved on the sheet: U1
